File: KICAD/kicad_chat-souris.kicad_pcb (KiCad board)
At the start: 2 copper layers, 7 parts, among them IC201 STM32G070RBT6, J201 ST/link connector, U301 MP1475, U302 MIC5317-3.3xM5, U401 ZXBM5210-S, U402 ZXBM5210-S, U501 MPU-6050

Commit message: Completed schematics
Parts:
- added C201: 0.1uF, Capacitor_SMD:C_0603_1608Metric, F.Cu at (75.1, 67.3)
- added C202: 0.1uF, Capacitor_SMD:C_0603_1608Metric, F.Cu at (75.1, 69.8)
- added C203: 0.1uF, Capacitor_SMD:C_0603_1608Metric, F.Cu at (75.1, 72.3)
- added C204: 10pF, Capacitor_SMD:C_0603_1608Metric, F.Cu at (75.1, 74.8)
- added C205: 10pF, Capacitor_SMD:C_0603_1608Metric, F.Cu at (75.1, 77.3)
- added C301: 22uF, Capacitor_SMD:C_0603_1608Metric, F.Cu at (62.7, 127.2)
- added C302: 0.1uF, Capacitor_SMD:C_0603_1608Metric, F.Cu at (62.7, 129.7)
- added C303: 0.1uF, Capacitor_SMD:C_0603_1608Metric, F.Cu at (62.7, 132.2)
- added C304: 0.1uF, Capacitor_SMD:C_0603_1608Metric, F.Cu at (62.7, 134.7)
- added C305: 0.1uF, Capacitor_SMD:C_0603_1608Metric, F.Cu at (62.7, 137.2)
- added C306: 22uF, Capacitor_SMD:C_0603_1608Metric, F.Cu at (62.7, 139.7)
- added C307: 22uF, Capacitor_SMD:C_0603_1608Metric, F.Cu at (66.7, 127.2)
- added C308: 1uF, Capacitor_SMD:C_0603_1608Metric, F.Cu at (66.7, 129.7)
- added C309: 1uF, Capacitor_SMD:C_0603_1608Metric, F.Cu at (66.7, 132.2)
- added C401: 1uF, Capacitor_SMD:C_0603_1608Metric, F.Cu at (82.1, 96.4)
- added C402: 1uF, Capacitor_SMD:C_0603_1608Metric, F.Cu at (82.1, 98.9)
- added C403: 47nF, Capacitor_SMD:C_0603_1608Metric, F.Cu at (82.1, 101.4)
- added C404: 47nF, Capacitor_SMD:C_0603_1608Metric, F.Cu at (82.1, 103.9)
- added C405: 10uF, Capacitor_SMD:CP_Elec_5x5.4, F.Cu at (84.6, 113.6)
- added C406: 10uF, Capacitor_SMD:CP_Elec_5x5.4, F.Cu at (84.6, 120.5)
- added C407: 47nF, Capacitor_SMD:C_0603_1608Metric, F.Cu at (82.1, 106.4)
- added C408: 47nF, Capacitor_SMD:C_0603_1608Metric, F.Cu at (82.1, 109.0)
- added C501: 0.01nF, Capacitor_SMD:C_0603_1608Metric, F.Cu at (49.3, 80.8)
- added C502: 0.01uF, Capacitor_SMD:C_0603_1608Metric, F.Cu at (49.3, 83.4)
- added C503: 0.1uF, Capacitor_SMD:C_0603_1608Metric, F.Cu at (49.3, 85.9)
- added C504: 2.2nF, Capacitor_SMD:C_0603_1608Metric, F.Cu at (49.3, 88.4)
- added C801: 0.1µF, Capacitor_SMD:C_0603_1608Metric, F.Cu at (24.8, 112.0)
- added C802: 100n, Capacitor_SMD:C_0603_1608Metric, F.Cu at (24.8, 114.5)
- added C803: 100n, Capacitor_SMD:C_0603_1608Metric, F.Cu at (24.8, 117.0)
- added C804: 100nF, Capacitor_SMD:C_0603_1608Metric, F.Cu at (24.8, 119.5)
- added C805: 10µ, Capacitor_SMD:CP_Elec_5x5.4, F.Cu at (40.2, 135.3)
- added C806: 1µF, Capacitor_SMD:C_0603_1608Metric, F.Cu at (24.8, 122.0)
- added D201: green, LED_SMD:LED_0603_1608Metric, F.Cu at (80.4, 82.4)
- added D202: red, LED_SMD:LED_0603_1608Metric, F.Cu at (80.4, 85.0)
- added D301: blue, LED_SMD:LED_0603_1608Metric, F.Cu at (79.7, 140.8)
- added D801: LED, LED_SMD:LED_0603_1608Metric, F.Cu at (37.8, 140.0)
- added D802: D_Schottky, Diode_SMD:D_SMA, F.Cu at (48.8, 140.6)
- added F801: MF-NSML150/12-2, Fuse:Fuse_1206_3216Metric, F.Cu at (25.6, 135.8)
- added J202: Conn_01x07, Connector_PinSocket_2.54mm:PinSocket_1x07_P2.54mm_Vertical, F.Cu at (65.0, 68.4)
- added J301: power switch JST, Connector_JST:JST_XH_S3B-XH-A_1x03_P2.50mm_Horizontal, F.Cu at (76.2, 129.2)
- added J401: Conn_motor1, Connector_JST:JST_XH_S6B-XH-A_1x06_P2.50mm_Horizontal, F.Cu at (64.2, 98.5)
- added J402: Conn_motor2, Connector_JST:JST_XH_S6B-XH-A_1x06_P2.50mm_Horizontal, F.Cu at (64.2, 112.0)
- added J501: Conn_Bmp_1, Connector_JST:JST_XH_S2B-XH-A_1x02_P2.50mm_Horizontal, F.Cu at (26.3, 69.4)
- added J502: Conn_Bmp_2, Connector_JST:JST_XH_S2B-XH-A_1x02_P2.50mm_Horizontal, F.Cu at (35.8, 69.4)
- added J503: Conn_lidar, Connector_JST:JST_XH_S8B-XH-A_1x08_P2.50mm_Horizontal, F.Cu at (26.3, 82.9)
- added J504: Conn_Bmp_3, Connector_JST:JST_XH_S2B-XH-A_1x02_P2.50mm_Horizontal, F.Cu at (45.2, 69.4)
- added J505: Conn_Bmp_4, Connector_JST:JST_XH_S2B-XH-A_1x02_P2.50mm_Horizontal, F.Cu at (54.7, 69.4)
- added J604: Conn_bord1, Connector_JST:JST_XH_S3B-XH-A_1x03_P2.50mm_Horizontal, F.Cu at (26.3, 98.5)
- added J605: Conn_bord2, Connector_JST:JST_XH_S3B-XH-A_1x03_P2.50mm_Horizontal, F.Cu at (38.3, 98.5)
- added J606: Conn_bord3, Connector_JST:JST_XH_S3B-XH-A_1x03_P2.50mm_Horizontal, F.Cu at (50.2, 98.5)
- added J801: DC_Jack_ALIM, DCJack_footprint:WE_694102303002, F.Cu at (42.5, 127.5)
- added J802: NiMH_Conn, Connector_JST:JST_XH_S2B-XH-A_1x02_P2.50mm_Horizontal, F.Cu at (34.3, 114.0)
- added J803: Li-Ion_Conn, Connector_JST:JST_XH_S3B-XH-A_1x03_P2.50mm_Horizontal, F.Cu at (43.8, 114.0)
- added JP801: SolderJumper_3_Open, Jumper:SolderJumper-3_P2.0mm_Open_TrianglePad1.0x1.5mm, F.Cu at (26.3, 132.1)
- added L301: 4.7uH, Inductor_SMD:L_1008_2520Metric, F.Cu at (75.2, 141.3)
- added Q801: NMOS, Package_TO_SOT_SMD:SOT-23, F.Cu at (33.3, 126.5)
- added Q802: NMOS, Package_TO_SOT_SMD:SOT-23, F.Cu at (33.3, 130.9)
- added Q803: PMOS, Package_TO_SOT_SMD:SOT-23, F.Cu at (33.3, 135.4)
- added R201: 20k, Resistor_SMD:R_0603_1608Metric, F.Cu at (75.1, 79.8)
- added R202: 20k, Resistor_SMD:R_0603_1608Metric, F.Cu at (79.1, 67.3)
- added R203: 20k, Resistor_SMD:R_0603_1608Metric, F.Cu at (79.1, 69.8)
- added R204: 5, Resistor_SMD:R_0603_1608Metric, F.Cu at (79.1, 72.3)
- added R205: 65, Resistor_SMD:R_0603_1608Metric, F.Cu at (79.1, 74.8)
- added R206: 10, Resistor_SMD:R_0603_1608Metric, F.Cu at (79.1, 77.3)
- added R301: 10k, Resistor_SMD:R_0603_1608Metric, F.Cu at (66.7, 134.7)
- added R302: 100k, Resistor_SMD:R_0603_1608Metric, F.Cu at (66.7, 137.2)
- added R303: 20, Resistor_SMD:R_0603_1608Metric, F.Cu at (66.7, 139.7)
- added R304: 16k, Resistor_SMD:R_0603_1608Metric, F.Cu at (70.7, 127.2)
- added R305: 7.68k, Resistor_SMD:R_0603_1608Metric, F.Cu at (70.7, 129.7)
- added R306: 40.2k, Resistor_SMD:R_0603_1608Metric, F.Cu at (70.7, 132.2)
- added R307: 100, Resistor_SMD:R_0603_1608Metric, F.Cu at (70.7, 134.7)
- added R501: 10k, Resistor_SMD:R_0603_1608Metric, F.Cu at (49.3, 90.9)
- added R502: 10k, Resistor_SMD:R_0603_1608Metric, F.Cu at (53.3, 80.8)
- added R503: 10k, Resistor_SMD:R_0603_1608Metric, F.Cu at (53.3, 83.4)
- added R504: 10k, Resistor_SMD:R_0603_1608Metric, F.Cu at (53.3, 85.9)
- added R505: 4.7k, Resistor_SMD:R_0603_1608Metric, F.Cu at (53.3, 88.4)
- added R506: 4.7k, Resistor_SMD:R_0603_1608Metric, F.Cu at (53.3, 90.9)
- added R801: 2k, Resistor_SMD:R_0603_1608Metric, F.Cu at (24.8, 124.5)
- added R802: 100, Resistor_SMD:R_0603_1608Metric, F.Cu at (28.9, 112.0)
- added R803: 100, Resistor_SMD:R_0603_1608Metric, F.Cu at (28.9, 114.5)
- added R804: 100, Resistor_SMD:R_0603_1608Metric, F.Cu at (28.9, 117.0)
- added R805: 2k, Resistor_SMD:R_0603_1608Metric, F.Cu at (28.9, 119.5)
- added R806: 19.6k, Resistor_SMD:R_0603_1608Metric, F.Cu at (28.9, 122.0)
- added R_SENSE801: 0.2, Resistor_SMD:R_1206_3216Metric, F.Cu at (25.6, 139.1)
- added SW201: RESET, Button_Switch_SMD:SW_SPST_B3U-1000P, F.Cu at (70.2, 68.2)
- added SW202: BTN_1, Button_Switch_SMD:SW_SPST_B3U-1000P, F.Cu at (70.2, 72.6)
- added SW203: BTN_2, Button_Switch_SMD:SW_SPST_B3U-1000P, F.Cu at (70.2, 76.9)
- added SW204: BTN_3, Button_Switch_SMD:SW_SPST_B3U-1000P, F.Cu at (70.2, 81.3)
- added U701: ~, Connector_PinSocket_2.54mm:PinSocket_1x07_P2.54mm_Horizontal, F.Cu at (95.5, 68.3)
- added U801: LTC1731ES8-8_4, Package_SO:SO-8_3.9x4.9mm_P1.27mm, F.Cu at (48.9, 135.1)
- added U802: ~, Package_SO:MSOP-8_3x3mm_P0.65mm, F.Cu at (26.5, 128.0)
- added Y201: Crystal, Crystal:Crystal_SMD_3225-4Pin_3.2x2.5mm, F.Cu at (75.7, 83.3)
- U401, U402: footprint Package_SO:SOIC-8_3.9x4.9mm_P1.27mm -> Package_SO:SOIC-8-1EP_3.9x4.9mm_P1.27mm_EP2.62x3.51mm
