File: KICAD/kicad_chat-souris.kicad_pcb (KiCad board)
At the start: 2 copper layers, 99 parts, among them IC201 STM32G070RBT6, J201 ST/link connector, J202 Conn_01x07, J301 power switch JST, J401 Conn_motor1, J402 Conn_motor2, J501 Conn_Bmp_1, J502 Conn_Bmp_2, J503 Conn_lidar, J504 Conn_Bmp_3, J505 Conn_Bmp_4, J604 Conn_bord1, J605 Conn_bord2, J606 Conn_bord3, J801 DC_Jack_ALIM, J802 NiMH_Conn, J803 Li-Ion_Conn, Q801 NMOS, Q802 NMOS, Q803 PMOS, SW201 RESET, SW202 BTN_1, SW203 BTN_2, SW204 BTN_3, U301 MP1475, U302 MIC5317-3.3xM5, U401 ZXBM5210-S, U402 ZXBM5210-S, U501 MPU-6050, U801 LTC1731ES8-8_4, Y201 Crystal

Commit message: PCB finalized
Parts:
- removed J202: Conn_01x07, Connector_PinSocket_2.54mm:PinSocket_1x07_P2.54mm_Vertical
- removed J501: Conn_Bmp_1, Connector_JST:JST_XH_S2B-XH-A_1x02_P2.50mm_Horizontal
- removed J502: Conn_Bmp_2, Connector_JST:JST_XH_S2B-XH-A_1x02_P2.50mm_Horizontal
- removed J604: Conn_bord1, Connector_JST:JST_XH_S3B-XH-A_1x03_P2.50mm_Horizontal
- removed J605: Conn_bord2, Connector_JST:JST_XH_S3B-XH-A_1x03_P2.50mm_Horizontal
- removed J606: Conn_bord3, Connector_JST:JST_XH_S3B-XH-A_1x03_P2.50mm_Horizontal
- added C1: 470n, Capacitor_SMD:C_0603_1608Metric, F.Cu at (128.5, 93.5)
- added C2: 4.7µ, Capacitor_SMD:C_0603_1608Metric, F.Cu at (128.6, 95.2)
- added C505: 4.7µ, Capacitor_SMD:CP_Elec_5x5.4, F.Cu at (114.3, 98.7)
- added D302: blue, LED_SMD:LED_0603_1608Metric, F.Cu at (150.1, 102.3)
- added D303: blue, LED_SMD:LED_0603_1608Metric, F.Cu at (157.8, 102.3)
- added FWD: Pin_D1.0mm_L10.0mm_LooseFit, Connector_Pin:Pin_D1.0mm_L10.0mm_LooseFit, F.Cu at (169.1, 108.7)
- added FWD: Pin_D1.0mm_L10.0mm_LooseFit, Connector_Pin:Pin_D1.0mm_L10.0mm_LooseFit, F.Cu at (169.1, 94.7)
- added G***: LOGO, IMAGE_PROJET:Logo_ENSEA, F.Cu at (105.4, 104.5)
- added G***: LOGO, IMAGE_PROJET:Logo_ENSEA, B.Cu at (113.6, 64.2)
- added G1: LOGO, IMAGE_PROJET:CHAT_SOURIE, B.Cu at (145.6, 84.2)
- added J2: Conn_02x07_Counter_Clockwise, Connector_PinHeader_2.54mm:PinHeader_2x07_P2.54mm_Vertical, F.Cu at (127.7, 52.4)
- added J302: 3V3, Connector_PinHeader_2.54mm:PinHeader_1x01_P2.54mm_Vertical, F.Cu at (144.1, 99.0)
- added J303: 5V, Connector_PinHeader_2.54mm:PinHeader_1x01_P2.54mm_Vertical, F.Cu at (151.8, 99.0)
- added J304: V_BAT, Connector_PinHeader_2.54mm:PinHeader_1x01_P2.54mm_Vertical, F.Cu at (159.6, 99.0)
- added J305: GND, Connector_PinHeader_2.54mm:PinHeader_1x01_P2.54mm_Vertical, F.Cu at (166.3, 117.2)
- added J506: SDA, Connector_PinHeader_2.54mm:PinHeader_1x01_P2.54mm_Vertical, F.Cu at (135.6, 74.0)
- added J507: SCL, Connector_PinHeader_2.54mm:PinHeader_1x01_P2.54mm_Vertical, F.Cu at (124.8, 74.2)
- added J601: Conn_bord1, Connector_JST:JST_XH_S3B-XH-A_1x03_P2.50mm_Horizontal, F.Cu at (112.5, 116.0)
- added J602: Conn_bord2, Connector_JST:JST_XH_S3B-XH-A_1x03_P2.50mm_Horizontal, F.Cu at (140.0, 55.0)
- added R1: R_Small, Resistor_SMD:R_0603_1608Metric, F.Cu at (127.6, 58.4)
- added R2: R_Small, Resistor_SMD:R_0603_1608Metric, F.Cu at (125.1, 58.4)
- added R3: R_Small, Resistor_SMD:R_0603_1608Metric, F.Cu at (122.5, 58.4)
- added R308: 50, Resistor_SMD:R_0603_1608Metric, F.Cu at (151.7, 102.3)
- added R309: 270, Resistor_SMD:R_0603_1608Metric, F.Cu at (159.4, 102.3)
- added R4: R_Small, Resistor_SMD:R_0603_1608Metric, F.Cu at (120.0, 58.4)
- added R5: R_Small, Resistor_SMD:R_0603_1608Metric, F.Cu at (117.5, 58.4)
- added R6: R_Small, Resistor_SMD:R_0603_1608Metric, F.Cu at (115.0, 58.4)
- added R7: R_Small, Resistor_SMD:R_0603_1608Metric, F.Cu at (112.5, 58.4)
- added REF**: MountingHole_3.2mm_M3_Pad_Via, MountingHole:MountingHole_3.2mm_M3_Pad_Via, F.Cu at (105.0, 55.0)
- added REF**: MountingHole_3.2mm_M3_Pad_Via, MountingHole:MountingHole_3.2mm_M3_Pad_Via, F.Cu at (185.0, 115.0)
- added REF**: MountingHole_3.2mm_M3_Pad_Via, MountingHole:MountingHole_3.2mm_M3_Pad_Via, F.Cu at (185.0, 55.0)
- added REF**: MountingHole_3.2mm_M3_Pad_Via, MountingHole:MountingHole_3.2mm_M3_Pad_Via, F.Cu at (105.0, 115.0)
- added REV: Pin_D1.0mm_L10.0mm_LooseFit, Connector_Pin:Pin_D1.0mm_L10.0mm_LooseFit, F.Cu at (175.3, 108.7)
- added REV: Pin_D1.0mm_L10.0mm_LooseFit, Connector_Pin:Pin_D1.0mm_L10.0mm_LooseFit, F.Cu at (175.3, 94.7)
- added locked: Conn_Bmp_1, Connector_JST:JST_XH_S2B-XH-A_1x02_P2.50mm_Horizontal, F.Cu at (129.2, 115.8)
- added locked: Conn_Bmp_2, Connector_JST:JST_XH_S2B-XH-A_1x02_P2.50mm_Horizontal, F.Cu at (148.2, 115.8)
- added locked: Conn_bord3, Connector_JST:JST_XH_S3B-XH-A_1x03_P2.50mm_Horizontal, F.Cu at (172.5, 116.0)
- D201: value green -> led_green
- D202: value red -> led_red
- J801: value DC_Jack_ALIM -> 694102303002; footprint DCJack_footprint:WE_694102303002 -> Connector_BarrelJack:BarrelJack_Wuerth_6941xx301002
- JP801: value SolderJumper_3_Open -> SolderJumper
- U302: value MIC5317-3.3xM5 -> MIC5317-3.3v
- U401: value ZXBM5210-S -> ZXBM5210-S_1; footprint Package_SO:SOIC-8-1EP_3.9x4.9mm_P1.27mm_EP2.62x3.51mm -> Package_SO:Diodes_SO-8EP
- U402: value ZXBM5210-S -> ZXBM5210-S_2; footprint Package_SO:SOIC-8-1EP_3.9x4.9mm_P1.27mm_EP2.62x3.51mm -> Package_SO:Diodes_SO-8EP
- U701: footprint Connector_PinSocket_2.54mm:PinSocket_1x07_P2.54mm_Horizontal -> Connector_PinSocket_2.54mm:PinSocket_1x06_P2.54mm_Vertical
- moved R_SENSE801 165.8 mm to (176.2, 69.8), turned to 90 degrees
- moved F801 161.6 mm to (168.3, 60.0), turned to 180 degrees
- moved C805 153.0 mm to (174.6, 62.0)
- moved Q803 152.9 mm to (169.1, 65.2)
- moved R801 151.9 mm to (169.0, 76.7)
- moved R806 151.6 mm to (172.5, 73.6), turned to 180 degrees
- moved J801 151.1 mm to (180.5, 66.0), turned to 90 degrees
- moved JP801 150.0 mm to (158.3, 60.7)
- moved C806 147.8 mm to (165.5, 76.7), turned to 180 degrees
- moved D801 147.1 mm to (169.0, 73.6)
- moved D802 146.1 mm to (179.6, 75.5), turned to 90 degrees
- moved C801 145.8 mm to (165.5, 73.6), turned to 180 degrees
- moved J802 143.4 mm to (165.0, 55.0), turned to 180 degrees
- moved U802 142.0 mm to (156.3, 70.3), turned to 90 degrees
- moved C804 141.8 mm to (159.3, 74.3), turned to -90 degrees
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Connections:
- net Net-(J401-Pin_1) renamed /Drivers and motors connectors/MOT1_OUT1
- net Net-(J401-Pin_6) renamed /Drivers and motors connectors/MOT1_OUT2
- net Net-(J402-Pin_1) renamed /Drivers and motors connectors/MOT2_OUT1
- net Net-(J402-Pin_6) renamed /Drivers and motors connectors/MOT2_OUT2
- net Net-(Q801-G) renamed /Alimentation/BMS/Secu_Dout
- net Net-(Q802-G) renamed /Alimentation/BMS/Secu_Vout
- net Net-(U301-FB) renamed /Alimentation/BUCK_FB
- net Net-(U301-SW) renamed /Alimentation/BUCK_SW
- net Net-(U802-Sense) renamed /Alimentation/BMS/Secu_Sense
- net Net-(U802-V-) renamed /Alimentation/BMS/Secu_V-
- net Net-(U802-VDD) renamed /Alimentation/BMS/Secu_VDD
- net Net-(U802-Vc) renamed /Alimentation/BMS/Secu_Vc
- D301 pad 2: +5V -> +3V3
- IC201 pad 3: /STM32/LIDAR_MOTOR_ENABLE -> /STM32/LIDAR_MESURE_ENABLE
- IC201 pad 33: /STM32/Bordure_1 -> /STM32/Bumper_3
- IC201 pad 34: /STM32/Bordure_2 -> /STM32/Bumper_4
- IC201 pad 38: /STM32/Bumper_1 -> /STM32/Bumper_2
- IC201 pad 39: /STM32/Bumper_2 -> /STM32/Bumper_1
- IC201 pad 4: /STM32/LIDAR_MESURE_ENABLE -> /STM32/LIDAR_MOTOR_ENABLE
- IC201 pad 40: /STM32/Bumper_3 -> /STM32/Bordure_1
- IC201 pad 41: /STM32/Bumper_4 -> /STM32/Bordure_2
- J201 pad 3: +3.3V -> +3V3
- J801 pad 3: (no net) -> GND
- J802 pad 1: NiMh+ -> GND
- J802 pad 2: GND -> NiMh+
- J803 pad 1: Li_Ion+ -> Li_Ion-
- J803 pad 3: Li_Ion- -> Li_Ion+
- R501 pad 2: +3.3V -> +3V3
- R502 pad 2: +3.3V -> +3V3
- R503 pad 2: +3.3V -> +3V3
- R504 pad 2: +3.3V -> +3V3
- U401 pad 9: (no net) -> GND
- U402 pad 9: (no net) -> GND
- Y201 pad 2: Net-(C205-Pad1) -> GND
- Y201 pad 3: (no net) -> Net-(C205-Pad1)
- Y201 pad 4: (no net) -> GND
Routing:
- net GND: track 0.00 -> 165.6 mm, vias 0 -> 38
- net +3V3: track 0.00 -> 155.1 mm, vias 0 -> 14
- net /Drivers and motors connectors/MOTOR_2_REV: track 0.00 -> 82.4 mm
- net /STM32/Bordure_3: track 0.00 -> 74.1 mm, vias 0 -> 1
- net /Drivers and motors connectors/MOTOR_2_FWD: track 0.00 -> 73.0 mm
- net /STM32/Bordure_1: track 0.00 -> 67.6 mm, vias 0 -> 1
- net /Drivers and motors connectors/MOTOR_1_REV: track 0.00 -> 65.5 mm, vias 0 -> 2
- net /Drivers and motors connectors/ENCODER_1_A: track 0.00 -> 61.8 mm, vias 0 -> 1
- net /STM32/Bumper_1: track 0.00 -> 60.4 mm, vias 0 -> 1
- net /STM32/Bumper_4: track 0.00 -> 59.6 mm, vias 0 -> 1
- net /Drivers and motors connectors/MOTOR_1_FWD: track 0.00 -> 59.3 mm, vias 0 -> 2
- net /Drivers and motors connectors/ENCODER_1_B: track 0.00 -> 58.4 mm, vias 0 -> 1
- net /Drivers and motors connectors/ENCODER_2_A: track 0.00 -> 58.1 mm, vias 0 -> 1
- net /Drivers and motors connectors/ENCODER_2_B: track 0.00 -> 57.8 mm, vias 0 -> 1
- net /STM32/Bumper_2: track 0.00 -> 54.5 mm, vias 0 -> 1
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- added copper zone on In1.Cu, net +3V3
- added copper zone on In1.Cu, net +5V
- added copper zone on In1.Cu, net +BATT
- added copper zone on B.Cu, net /Drivers and motors connectors/MOT1_OUT1
- added copper zone on F.Cu, net /Drivers and motors connectors/MOT1_OUT2
- added copper zone on B.Cu, net /Drivers and motors connectors/MOT2_OUT1
- added copper zone on F.Cu, net /Drivers and motors connectors/MOT2_OUT2
- added copper zone on In2.Cu, net GND
Other:
- board outline added: 90 x 70 mm
- copper layers 2 -> 4
- board text added: "+3V3"
- board text added: "+5V"
- board text added: "+BAT"
- board text added: "1"
- board text added: "2"
- board text added: "3"
- board text added: "4"
- board text added: "BMS"
- board text added: "BORD_1"
- board text added: "BORD_2"
- board text added: "BORD_3"
- board text added: "BUMPERS"
- board text added: "BUTTON"
- board text added: "Fuse"
- board text added: "GND"
- board text added: "GPIO_D"
- board text added: "HC05"
- board text added: "LED_G"
- board text added: "LED_R"
- board text added: "LIDAR"
- board text added: "Li_Ion"
- board text added: "MPU"
- board text added: "Maxime PICHERY Baptiste RODIER Martina VAN DE MOOSDJIK Paul-Etienne RETAUX"
- board text added: "Motor Driver"
- board text added: "NiMh"
- board text added: "PWR_CONV"
- board text added: "Project : Robot Chat Souris ENSEA 3A ESE 2023-2024"
- board text added: "RST"
- board text added: "R_Sense"
- board text added: "SCL"
- board text added: "SDA"
- board text added: "STLink"
- board text added: "STM32"
- board text added: "Switch"
- board text added: "USER"
