File: KICAD/Capteur de bordure.kicad_sch (KiCad schematic)
At the start: 12 parts, among them J301 Conn_01x09, J302 Conn_01x09, J303 Conn_01x09

Commit message: update schematics
Parts:
- C301, C302, C303, C304, C305, C306: footprint (none) -> Capacitor_SMD:C_0603_1608Metric
Changed lines of the file:
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@@
       (effects (font (size 1.27 1.27)) (justify left))
     )
-    (property "Footprint" "" (at 46.99 93.98 0)
+    (property "Footprint" "Capacitor_SMD:C_0603_1608Metric" (at 46.99 93.98 0)
       (effects (font (size 1.27 1.27)) hide)
     )
@@
       (effects (font (size 1.27 1.27)) (justify left))
     )
-    (property "Footprint" "" (at 36.83 137.16 0)
+    (property "Footprint" "Capacitor_SMD:C_0603_1608Metric" (at 36.83 137.16 0)
       (effects (font (size 1.27 1.27)) hide)
     )
@@
       (effects (font (size 1.27 1.27)) (justify left))
     )
-    (property "Footprint" "" (at 36.83 99.06 0)
+    (property "Footprint" "Capacitor_SMD:C_0603_1608Metric" (at 36.83 99.06 0)
       (effects (font (size 1.27 1.27)) hide)
     )
@@
       (effects (font (size 1.27 1.27)) (justify left))
     )
-    (property "Footprint" "" (at 46.99 132.08 0)
+    (property "Footprint" "Capacitor_SMD:C_0603_1608Metric" (at 46.99 132.08 0)
       (effects (font (size 1.27 1.27)) hide)
     )
@@
       (effects (font (size 1.27 1.27)) (justify left))
     )
-    (property "Footprint" "" (at 46.99 168.91 0)
+    (property "Footprint" "Capacitor_SMD:C_0603_1608Metric" (at 46.99 168.91 0)
       (effects (font (size 1.27 1.27)) hide)
     )
@@
       (effects (font (size 1.27 1.27)) (justify left))
     )
-    (property "Footprint" "" (at 36.83 173.99 0)
-      (effects (font (size 1.27 1.27)) hide)
-    )
+    (property "Footprint" "Capacitor_SMD:C_0603_1608Metric" (at 36.83 173.99 0)
+      (effects (font (size 1.27 1.27)) hide)
+    )

Commit message: Completed schematics
Parts:
- removed C301, C302, C303, C304, C305, C306: 100 nF, Capacitor_SMD:C_0603_1608Metric, symbol Device:C_Small
- removed J301, J302, J303: Conn_01x09, symbol Connector_Generic:Conn_01x09
- removed R301, R302, R303: 4.3 Ohm, symbol Device:R_Small
- added J601: Conn_bord1, Connector_JST:JST_XH_S3B-XH-A_1x03_P2.50mm_Horizontal, symbol Connector_Generic:Conn_01x03
- added J602: Conn_bord2, Connector_JST:JST_XH_S3B-XH-A_1x03_P2.50mm_Horizontal, symbol Connector_Generic:Conn_01x03
- added J603: Conn_bord3, Connector_JST:JST_XH_S3B-XH-A_1x03_P2.50mm_Horizontal, symbol Connector_Generic:Conn_01x03
Connections:
- net +3.3V: now also J601.2 (Pin_2), J602.2 (Pin_2), J603.2 (Pin_2)
- net Bord_1_out: now also J601.3 (Pin_3)
- net Bord_2_out: now also J602.3 (Pin_3)
- net Bord_3_out: now also J603.3 (Pin_3)
- net GND: now also J601.1 (Pin_1), J602.1 (Pin_1), J603.1 (Pin_1)
Other:
- note removed: "Branchement connecteur JST-Capteur de bordure: JST | Capteur 1->1 2->3 3->2 4->4 5->7 6->11 7->12 8->13 9->14"

Commit message: PCB finalized
Connections:
- net +3.3V renamed +3V3
Changed lines of the file:
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@@
 (kicad_sch (version 20230121) (generator eeschema)
   (paper "A4")
+  (wire (pts (xy 78.74 90.17) (xy 80.01 90.17))
+    (stroke (width 0) (type default))
+  )
+  (wire (pts (xy 41.91 90.17) (xy 43.18 90.17))
+    (stroke (width 0) (type default))
+  )
+  (wire (pts (xy 115.57 90.17) (xy 116.84 90.17))
+    (stroke (width 0) (type default))
+  )
   (text "Capteur de bordure 1" (at 57.15 83.82 0)
     (effects (font (size 1.27 1.27)) (justify right bottom))
@@
     )
   )
-  (symbol (lib_id "power:+3.3V") (at 116.84 90.17 90) (unit 1)
-    (in_bom yes) (on_board yes) (dnp no) (fields_autoplaced)
-    (property "Reference" "#PWR0306" (at 120.65 90.17 0)
-      (effects (font (size 1.27 1.27)) hide)
-    )
-    (property "Value" "+3.3V" (at 113.03 90.17 90)
-      (effects (font (size 1.27 1.27)) (justify left))
-    )
-    (property "Footprint" "" (at 116.84 90.17 0)
-      (effects (font (size 1.27 1.27)) hide)
-    )
-    (property "Datasheet" "" (at 116.84 90.17 0)
-      (effects (font (size 1.27 1.27)) hide)
-    )
-    (pin "1")
-    (instances
-      (project "projet"
-        (path "/72843e5b-039f-43c6-ac6b-21bc38672670/0c63e019-08e8-4abf-82ad-8b25334b9bc2/acc32a84-b93a-4520-8f59-7d8bc453a92b"
-          (reference "#PWR0306") (unit 1)
-        )
-      )
-      (project "kicad_chat-souris"
-        (path "/b1ddc66d-dbe7-4cff-b97f-1f0ce7ceeee4/1d2079b7-f9a0-4747-bb76-648b078e7186/1be7610a-d812-4888-a929-417febc6b201"
-          (reference "#PWR0606") (unit 1)
-        )
-      )
-    )
-  )
-  (symbol (lib_id "power:+3.3V") (at 43.18 90.17 90) (unit 1)
-    (in_bom yes) (on_board yes) (dnp no) (fields_autoplaced)
-    (property "Reference" "#PWR0306" (at 46.99 90.17 0)
-      (effects (font (size 1.27 1.27)) hide)
-    )
-    (property "Value" "+3.3V" (at 39.37 90.17 90)
-      (effects (font (size 1.27 1.27)) (justify left))
-    )
-    (property "Footprint" "" (at 43.18 90.17 0)
-      (effects (font (size 1.27 1.27)) hide)
-    )
-    (property "Datasheet" "" (at 43.18 90.17 0)
-      (effects (font (size 1.27 1.27)) hide)
-    )
-    (pin "1")
-    (instances
-      (project "projet"
-        (path "/72843e5b-039f-43c6-ac6b-21bc38672670/0c63e019-08e8-4abf-82ad-8b25334b9bc2/acc32a84-b93a-4520-8f59-7d8bc453a92b"
-          (reference "#PWR0306") (unit 1)
-        )
-      )
-      (project "kicad_chat-souris"
-        (path "/b1ddc66d-dbe7-4cff-b97f-1f0ce7ceeee4/1d2079b7-f9a0-4747-bb76-648b078e7186/1be7610a-d812-4888-a929-417febc6b201"
-          (reference "#PWR0602") (unit 1)
-        )
-      )
-    )
-  )
-  (symbol (lib_id "power:+3.3V") (at 80.01 90.17 90) (unit 1)
-    (in_bom yes) (on_board yes) (dnp no) (fields_autoplaced)
-    (property "Reference" "#PWR0306" (at 83.82 90.17 0)
-      (effects (font (size 1.27 1.27)) hide)
-    )
-    (property "Value" "+3.3V" (at 76.2 90.17 90)
-      (effects (font (size 1.27 1.27)) (justify left))
-    )
-    (property "Footprint" "" (at 80.01 90.17 0)
-      (effects (font (size 1.27 1.27)) hide)
-    )
-    (property "Datasheet" "" (at 80.01 90.17 0)
-      (effects (font (size 1.27 1.27)) hide)
-    )
-    (pin "1")
-    (instances
-      (project "projet"
-        (path "/72843e5b-039f-43c6-ac6b-21bc38672670/0c63e019-08e8-4abf-82ad-8b25334b9bc2/acc32a84-b93a-4520-8f59-7d8bc453a92b"
-          (reference "#PWR0306") (unit 1)
-        )
-      )
-      (project "kicad_chat-souris"
-        (path "/b1ddc66d-dbe7-4cff-b97f-1f0ce7ceeee4/1d2079b7-f9a0-4747-bb76-648b078e7186/1be7610a-d812-4888-a929-417febc6b201"
-          (reference "#PWR0604") (unit 1)
-        )
-      )
+  (symbol (lib_id "power:+3V3") (at 115.57 90.17 90) (unit 1)
+    (in_bom yes) (on_board yes) (dnp no) (fields_autoplaced)
+    (property "Reference" "#PWR01" (at 119.38 90.17 0)
+      (effects (font (size 1.27 1.27)) hide)
+    )
+    (property "Value" "+3V3" (at 111.76 90.17 90)
+      (effects (font (size 1.27 1.27)) (justify left))
+    )
+    (property "Footprint" "" (at 115.57 90.17 0)
+      (effects (font (size 1.27 1.27)) hide)
+    )
+    (property "Datasheet" "" (at 115.57 90.17 0)
+      (effects (font (size 1.27 1.27)) hide)
+    )
+    (pin "1")
+    (instances
+      (project "kicad_chat-souris"
+        (path "/b1ddc66d-dbe7-4cff-b97f-1f0ce7ceeee4/1d2079b7-f9a0-4747-bb76-648b078e7186"
+          (reference "#PWR01") (unit 1)
+        )
+        (path "/b1ddc66d-dbe7-4cff-b97f-1f0ce7ceeee4/1d2079b7-f9a0-4747-bb76-648b078e7186/1be7610a-d812-4888-a929-417febc6b201"
+          (reference "#PWR08") (unit 1)
+        )
+      )
+    )
+  )
+  (symbol (lib_id "power:+3V3") (at 78.74 90.17 90) (unit 1)
+    (in_bom yes) (on_board yes) (dnp no) (fields_autoplaced)
+    (property "Reference" "#PWR01" (at 82.55 90.17 0)
+      (effects (font (size 1.27 1.27)) hide)
+    )
+    (property "Value" "+3V3" (at 74.93 90.17 90)
+      (effects (font (size 1.27 1.27)) (justify left))
+    )
+    (property "Footprint" "" (at 78.74 90.17 0)
+      (effects (font (size 1.27 1.27)) hide)
+    )
+    (property "Datasheet" "" (at 78.74 90.17 0)
+      (effects (font (size 1.27 1.27)) hide)
+    )
+    (pin "1")
+    (instances
+      (project "kicad_chat-souris"
+        (path "/b1ddc66d-dbe7-4cff-b97f-1f0ce7ceeee4/1d2079b7-f9a0-4747-bb76-648b078e7186"
+          (reference "#PWR01") (unit 1)
+        )
+        (path "/b1ddc66d-dbe7-4cff-b97f-1f0ce7ceeee4/1d2079b7-f9a0-4747-bb76-648b078e7186/1be7610a-d812-4888-a929-417febc6b201"
+          (reference "#PWR07") (unit 1)
+        )
+      )
+    )
+  )
+  (symbol (lib_id "power:+3V3") (at 41.91 90.17 90) (unit 1)
+    (in_bom yes) (on_board yes) (dnp no) (fields_autoplaced)
+    (property "Reference" "#PWR01" (at 45.72 90.17 0)
+      (effects (font (size 1.27 1.27)) hide)
+    )
+    (property "Value" "+3V3" (at 38.1 90.17 90)
+      (effects (font (size 1.27 1.27)) (justify left))
+    )
+    (property "Footprint" "" (at 41.91 90.17 0)
+      (effects (font (size 1.27 1.27)) hide)
+    )
+    (property "Datasheet" "" (at 41.91 90.17 0)
+      (effects (font (size 1.27 1.27)) hide)
+    )
+    (pin "1")
+    (instances
+      (project "kicad_chat-souris"
+        (path "/b1ddc66d-dbe7-4cff-b97f-1f0ce7ceeee4/1d2079b7-f9a0-4747-bb76-648b078e7186"
+          (reference "#PWR01") (unit 1)
+        )
+        (path "/b1ddc66d-dbe7-4cff-b97f-1f0ce7ceeee4/1d2079b7-f9a0-4747-bb76-648b078e7186/1be7610a-d812-4888-a929-417febc6b201"
+          (reference "#PWR06") (unit 1)
+        )
+      )
