File: KICAD/STM32.kicad_sch (KiCad schematic)
At the start: 21 parts, among them IC201 STM32G070RBT6, J202 Conn_01x07, J301 ST/link connector, SW201 RESET, SW202 BTN_1, SW203 BTN_2, SW204 BTN_3, Y201 Crystal

Commit message: update schematics
Parts:
- C201, C202, C203, C204, C205: footprint (none) -> Capacitor_SMD:C_0603_1608Metric
- D601, D603: footprint (none) -> LED_SMD:LED_0603_1608Metric
Changed lines of the file:
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@@
       (effects (font (size 1.27 1.27)) (justify left))
     )
-    (property "Footprint" "" (at 45.72 181.61 0)
+    (property "Footprint" "Capacitor_SMD:C_0603_1608Metric" (at 45.72 181.61 0)
       (effects (font (size 1.27 1.27)) hide)
     )
@@
       (effects (font (size 1.27 1.27)))
     )
-    (property "Footprint" "" (at 124.46 163.83 90)
+    (property "Footprint" "LED_SMD:LED_0603_1608Metric" (at 124.46 163.83 90)
       (effects (font (size 1.27 1.27)) hide)
     )
@@
       (effects (font (size 1.27 1.27)) (justify left))
     )
-    (property "Footprint" "" (at 45.72 153.67 0)
+    (property "Footprint" "Capacitor_SMD:C_0603_1608Metric" (at 45.72 153.67 0)
       (effects (font (size 1.27 1.27)) hide)
     )
@@
       (effects (font (size 1.27 1.27)))
     )
-    (property "Footprint" "" (at 254 112.0648 0)
+    (property "Footprint" "Capacitor_SMD:C_0603_1608Metric" (at 254 112.0648 0)
       (effects (font (size 1.27 1.27)) hide)
     )
@@
       (effects (font (size 1.27 1.27)) (justify left))
     )
-    (property "Footprint" "" (at 45.72 167.64 0)
+    (property "Footprint" "Capacitor_SMD:C_0603_1608Metric" (at 45.72 167.64 0)
       (effects (font (size 1.27 1.27)) hide)
     )
@@
       (effects (font (size 1.27 1.27)))
     )
-    (property "Footprint" "" (at 113.03 163.83 90)
+    (property "Footprint" "LED_SMD:LED_0603_1608Metric" (at 113.03 163.83 90)
       (effects (font (size 1.27 1.27)) hide)
     )
@@
       (effects (font (size 1.27 1.27)))
     )
-    (property "Footprint" "" (at 254 122.2248 0)
-      (effects (font (size 1.27 1.27)) hide)
-    )
+    (property "Footprint" "Capacitor_SMD:C_0603_1608Metric" (at 254 122.2248 0)
+      (effects (font (size 1.27 1.27)) hide)
+    )

Commit message: Completed schematics
Parts:
- D601: value green -> led_green
- D603: value red -> led_red
- J202: value Conn_01x07 -> GPIOD; footprint (none) -> Connector_PinSocket_2.54mm:PinSocket_1x07_P2.54mm_Vertical
- R201, R202, R203, R206: footprint (none) -> Resistor_SMD:R_0603_1608Metric
- R601: value R_Small -> 5; footprint (none) -> Resistor_SMD:R_0603_1608Metric
- R603: value R_Small -> 65; footprint (none) -> Resistor_SMD:R_0603_1608Metric
- SW201, SW202, SW203, SW204: footprint (none) -> Button_Switch_SMD:SW_SPST_B3U-1000P
- Y201: footprint (none) -> Crystal:Crystal_SMD_3225-4Pin_3.2x2.5mm
Changed lines of the file:
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@@
   (junction (at 45.72 149.86) (diameter 0) (color 0 0 0 0)
+  )
+  (junction (at 222.25 76.2) (diameter 0) (color 0 0 0 0)
   )
   (junction (at 222.25 86.36) (diameter 0) (color 0 0 0 0)
@@
       (effects (font (size 1.27 1.27)) (justify left))
     )
-    (property "Value" "R_Small" (at 105.41 170.18 0)
+    (property "Value" "5" (at 107.95 170.18 0)
       (effects (font (size 1.27 1.27)) (justify left))
     )
-    (property "Footprint" "" (at 113.03 168.91 0)
+    (property "Footprint" "Resistor_SMD:R_0603_1608Metric" (at 113.03 168.91 0)
       (effects (font (size 1.27 1.27)) hide)
     )
@@
       (effects (font (size 1.27 1.27)))
     )
-    (property "Footprint" "" (at 33.02 137.16 0)
+    (property "Footprint" "Button_Switch_SMD:SW_SPST_B3U-1000P" (at 33.02 137.16 0)
       (effects (font (size 1.27 1.27)) hide)
     )
@@
       (effects (font (size 1.27 1.27)))
     )
-    (property "Footprint" "" (at 33.02 163.83 0)
+    (property "Footprint" "Button_Switch_SMD:SW_SPST_B3U-1000P" (at 33.02 163.83 0)
       (effects (font (size 1.27 1.27)) hide)
     )
@@
       (effects (font (size 1.27 1.27)))
     )
-    (property "Value" "red" (at 127 163.83 0)
+    (property "Value" "led_red" (at 127 163.83 0)
       (effects (font (size 1.27 1.27)))
     )
@@
       (effects (font (size 1.27 1.27)))
     )
-    (property "Footprint" "" (at 231.14 124.968 90)
+    (property "Footprint" "Resistor_SMD:R_0603_1608Metric" (at 231.14 124.968 90)
       (effects (font (size 1.27 1.27)) hide)
     )
@@
       (effects (font (size 1.27 1.27)))
     )
-    (property "Footprint" "" (at 55.88 149.86 0)
+    (property "Footprint" "Resistor_SMD:R_0603_1608Metric" (at 55.88 149.86 0)
       (effects (font (size 1.27 1.27)) hide)
     )
@@
       (effects (font (size 1.27 1.27)))
     )
-    (property "Footprint" "" (at 55.88 177.8 0)
+    (property "Footprint" "Resistor_SMD:R_0603_1608Metric" (at 55.88 177.8 0)
       (effects (font (size 1.27 1.27)) hide)
     )
@@
       (effects (font (size 1.27 1.27)))
     )
-    (property "Footprint" "" (at 33.02 177.8 0)
+    (property "Footprint" "Button_Switch_SMD:SW_SPST_B3U-1000P" (at 33.02 177.8 0)
       (effects (font (size 1.27 1.27)) hide)
     )
@@
       (effects (font (size 1.27 1.27)) (justify left))
     )
-    (property "Footprint" "" (at 243.84 118.11 0)
+    (property "Footprint" "Crystal:Crystal_SMD_3225-4Pin_3.2x2.5mm" (at 243.84 118.11 0)
       (effects (font (size 1.27 1.27)) hide)
     )
@@
       (effects (font (size 1.27 1.27)))
     )
-    (property "Footprint" "" (at 55.88 163.83 0)
+    (property "Footprint" "Resistor_SMD:R_0603_1608Metric" (at 55.88 163.83 0)
       (effects (font (size 1.27 1.27)) hide)
     )
@@
       (effects (font (size 1.27 1.27)))
     )
-    (property "Value" "green" (at 115.57 163.83 0)
+    (property "Value" "led_green" (at 115.57 163.83 0)
       (effects (font (size 1.27 1.27)))
     )
@@
         (path "/b1ddc66d-dbe7-4cff-b97f-1f0ce7ceeee4/a13fe5f2-f6e5-4a93-b768-5d6eb675b5fa"
           (reference "#PWR0209") (unit 1)
+        )
+      )
+    )
+  )
+  (symbol (lib_id "power:PWR_FLAG") (at 222.25 76.2 90) (unit 1)
+    (in_bom yes) (on_board yes) (dnp no) (fields_autoplaced)
+    (property "Reference" "#FLG0301" (at 220.345 76.2 0)
+      (effects (font (size 1.27 1.27)) hide)
+    )
+    (property "Value" "PWR_FLAG" (at 218.44 76.2 90)
+      (effects (font (size 1.27 1.27)) (justify left))
+    )
+    (property "Footprint" "" (at 222.25 76.2 0)
+      (effects (font (size 1.27 1.27)) hide)
+    )
+    (property "Datasheet" "~" (at 222.25 76.2 0)
+      (effects (font (size 1.27 1.27)) hide)
+    )
+    (pin "1")
+    (instances
+      (project "kicad_chat-souris"
+        (path "/b1ddc66d-dbe7-4cff-b97f-1f0ce7ceeee4/6a44a42c-5fbe-4248-b986-7ff99c499b51"
+          (reference "#FLG0301") (unit 1)
+        )
+        (path "/b1ddc66d-dbe7-4cff-b97f-1f0ce7ceeee4/a13fe5f2-f6e5-4a93-b768-5d6eb675b5fa"
+          (reference "#FLG0201") (unit 1)
         )
       )
@@
       (effects (font (size 1.27 1.27)) (justify right))
     )
-    (property "Value" "R_Small" (at 118.11 170.18 0)
+    (property "Value" "65" (at 118.11 170.18 0)
       (effects (font (size 1.27 1.27)) (justify right))
     )
-    (property "Footprint" "" (at 124.46 168.91 0)
+    (property "Footprint" "Resistor_SMD:R_0603_1608Metric" (at 124.46 168.91 0)
       (effects (font (size 1.27 1.27)) hide)
     )
@@
       (effects (font (size 1.27 1.27)) (justify left))
     )
-    (property "Value" "Conn_01x07" (at 246.38 52.07 0)
+    (property "Value" "GPIOD" (at 246.38 52.07 0)
       (effects (font (size 1.27 1.27)) (justify left))
     )
-    (property "Footprint" "" (at 243.84 50.8 0)
+    (property "Footprint" "Connector_PinSocket_2.54mm:PinSocket_1x07_P2.54mm_Vertical" (at 243.84 50.8 0)
       (effects (font (size 1.27 1.27)) hide)
     )
@@
       (effects (font (size 1.27 1.27)))
     )
-    (property "Footprint" "" (at 33.02 149.86 0)
-      (effects (font (size 1.27 1.27)) hide)
-    )
+    (property "Footprint" "Button_Switch_SMD:SW_SPST_B3U-1000P" (at 33.02 149.86 0)
+      (effects (font (size 1.27 1.27)) hide)
+    )

Commit message: PCB finalized
Parts:
- removed J202: GPIOD, Connector_PinSocket_2.54mm:PinSocket_1x07_P2.54mm_Vertical, symbol Connector_Generic:Conn_01x07
- added C1: 470n, Capacitor_SMD:C_0603_1608Metric, symbol Device:C_Small
- added C2: 4.7µ, Capacitor_SMD:C_0603_1608Metric, symbol Device:C_Small
- added J2: Conn_02x07_Counter_Clockwise, Connector_PinHeader_2.54mm:PinHeader_2x07_P2.54mm_Vertical, symbol Connector_Generic:Conn_02x07_Counter_Clockwise
- added R1, R2, R3, R4, R5, R6, R7: R_Small, Resistor_SMD:R_0603_1608Metric, symbol Device:R_Small
- Y201: symbol Device:Crystal -> Device:Crystal_GND24
Connections:
- net +3.3V is gone; now on net +3V3: J301.3 (Pin_3)
- net +3V3: now also C1.1, C2.1
- net Bordure_1: now also IC201.40 (PD8); no longer IC201.33 (PB13)
- net Bordure_2: now also IC201.41 (PD9); no longer IC201.34 (PB14)
- net Bumper_1: now also IC201.39 (PC7); no longer IC201.38 (PC6)
- net Bumper_2: now also IC201.38 (PC6); no longer IC201.39 (PC7)
- net Bumper_3: now also IC201.33 (PB13); no longer IC201.40 (PD8)
- net Bumper_4: now also IC201.34 (PB14); no longer IC201.41 (PD9)
- net GND: now also Y201.2, Y201.4, C1.2, C2.2, J2.1 (Pin_1), J2.11 (Pin_11), J2.13 (Pin_13), J2.3 (Pin_3), J2.5 (Pin_5), J2.7 (Pin_7), J2.9 (Pin_9)
- net LIDAR_MESURE_ENABLE: now also IC201.3 (PC13); no longer IC201.4 (PC14-OSC32_IN)
- net LIDAR_MOTOR_ENABLE: now also IC201.4 (PC14-OSC32_IN); no longer IC201.3 (PC13)
- net PD0: now also R5.1
- net PD1: now also R4.1
- net PD2: now also R1.1
- net PD3: now also R2.1
- net PD4: now also R3.1
- net PD5: now also R6.1
- net PD6: now also R7.1
- net at C205.1, R206.2: now also Y201.3; no longer Y201.2
- new net: J2.6 (Pin_6), R3.2
- new net: J2.12 (Pin_12), R6.2
- new net: J2.2 (Pin_2), R1.2
- new net: J2.8 (Pin_8), R4.2
- new net: J2.14 (Pin_14), R7.2
- new net: J2.10 (Pin_10), R5.2
- new net: J2.4 (Pin_4), R2.2
Other:
- note added: "J'ai inversé certain pin de Bordure et Bumper"
