File: KICAD/alimentation.kicad_sch (KiCad schematic)
At the start: 21 parts, among them SW301 POWER_switch, U301 MP1475, U302 MIC5317-3.3xM5

Commit message: update schematics
Parts:
- C301, C302, C303, C304, C305, C306, C307, C308, C309: footprint (none) -> Capacitor_SMD:C_0603_1608Metric
- D602: footprint (none) -> LED_SMD:LED_0603_1608Metric
Other:
- moved on the sheet: C301, C302, C303, C304, C305, C306, C307, C308, C309, D602, L301, R301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

Commit message: Completed schematics
Parts:
- removed SW301: POWER_switch, symbol Switch:SW_DP3T
- added J301: power switch JST, Connector_JST:JST_XH_S3B-XH-A_1x03_P2.50mm_Horizontal, symbol Connector_Generic:Conn_01x03
- L301: footprint (none) -> Inductor_SMD:L_1008_2520Metric
- R301, R302, R303, R304, R305, R306: footprint (none) -> Resistor_SMD:R_0603_1608Metric
- R602: value R_Small -> 100; footprint (none) -> Resistor_SMD:R_0603_1608Metric
- U302: value MIC5317-3.3xM5 -> MIC5317-3.3v
Connections:
- net +BATT: now also J301.2 (Pin_2)
- net BMS/BMS: now also J301.3 (Pin_3)
- no-connect marks 2 -> 1
Other:
- note added: "Pont diviseur de tension pour avoir la bonne tension de sortie"

Commit message: PCB finalized
Parts:
- added D602 (x2): blue, LED_SMD:LED_0603_1608Metric, symbol Device:LED_Small
- added J302: 3V3, Connector_PinHeader_2.54mm:PinHeader_1x01_P2.54mm_Vertical, symbol Connector:Conn_01x01_Pin
- added J303: 5V, Connector_PinHeader_2.54mm:PinHeader_1x01_P2.54mm_Vertical, symbol Connector:Conn_01x01_Pin
- added J304: V_BAT, Connector_PinHeader_2.54mm:PinHeader_1x01_P2.54mm_Vertical, symbol Connector:Conn_01x01_Pin
- added J305: GND, Connector_PinHeader_2.54mm:PinHeader_1x01_P2.54mm_Vertical, symbol Connector:Conn_01x01_Pin
- added R602: 50, Resistor_SMD:R_0603_1608Metric, symbol Device:R_Small
- added R602: 270, Resistor_SMD:R_0603_1608Metric, symbol Device:R_Small
Connections:
- net +3V3: now also D602.2 (A), J302.1 (Pin_1)
- net +5V: now also D602.2 (A), J303.1 (Pin_1); no longer D602.2 (A)
- net +BATT: now also D602.2 (A), J304.1 (Pin_1)
- net GND: now also J305.1 (Pin_1), R602.2, R602.2
- net BUCK_SW: now reaches C304.2, L301.1, U301.3 (SW)
- net BUCK_FB: now reaches R304.1, U301.8 (FB)
- new net: D602.1 (K), R602.1 (x2)
Other:
- note added: "Power status led"
- note removed: "5V Power status led"
- moved on the sheet: D602, R602
