File: KICAD/com.kicad_sch (KiCad schematic)
At the start: 1 part

Commit message: Completed schematics
Parts:
- U701: footprint (none) -> Connector_PinSocket_2.54mm:PinSocket_1x07_P2.54mm_Horizontal
Changed lines of the file:
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@@
       (effects (font (size 1.27 1.27)))
     )
-    (property "Footprint" "" (at 153.67 69.85 0)
+    (property "Footprint" "Connector_PinSocket_2.54mm:PinSocket_1x07_P2.54mm_Horizontal" (at 153.67 69.85 0)
       (effects (font (size 1.27 1.27)) hide)
     )

Commit message: PCB finalized
Parts:
- U701: footprint Connector_PinSocket_2.54mm:PinSocket_1x07_P2.54mm_Horizontal -> Connector_PinSocket_2.54mm:PinSocket_1x06_P2.54mm_Vertical
Changed lines of the file:
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@@
       (effects (font (size 1.27 1.27)))
     )
-    (property "Footprint" "Connector_PinSocket_2.54mm:PinSocket_1x07_P2.54mm_Horizontal" (at 153.67 69.85 0)
+    (property "Footprint" "Connector_PinSocket_2.54mm:PinSocket_1x06_P2.54mm_Vertical" (at 153.67 69.85 0)
       (effects (font (size 1.27 1.27)) hide)
     )
