File: KICAD/drivers.kicad_sch (KiCad schematic)
At the start: 12 parts, among them J401 Conn_motor1, J402 Conn_motor2, U401 ZXBM5210-S, U402 ZXBM5210-S

Commit message: update schematics
Parts:
- C401, C402, C403, C404, C405, C406, C407, C408: footprint (none) -> Capacitor_SMD:C_0603_1608Metric
Changed lines of the file:
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@@
       (effects (font (size 1.27 1.27)) (justify left))
     )
-    (property "Footprint" "" (at 101.6 72.39 0)
+    (property "Footprint" "Capacitor_SMD:C_0603_1608Metric" (at 101.6 72.39 0)
       (effects (font (size 1.27 1.27)) hide)
     )
@@
       (effects (font (size 1.27 1.27)) (justify left))
     )
-    (property "Footprint" "" (at 137.16 74.93 0)
+    (property "Footprint" "Capacitor_SMD:C_0603_1608Metric" (at 137.16 74.93 0)
       (effects (font (size 1.27 1.27)) hide)
     )
@@
       (effects (font (size 1.27 1.27)) (justify left))
     )
-    (property "Footprint" "" (at 134.62 135.89 0)
+    (property "Footprint" "Capacitor_SMD:C_0603_1608Metric" (at 134.62 135.89 0)
       (effects (font (size 1.27 1.27)) hide)
     )
@@
       (effects (font (size 1.27 1.27)) (justify left))
     )
-    (property "Footprint" "" (at 137.16 118.11 0)
+    (property "Footprint" "Capacitor_SMD:C_0603_1608Metric" (at 137.16 118.11 0)
       (effects (font (size 1.27 1.27)) hide)
     )
@@
       (effects (font (size 1.27 1.27)) (justify left))
     )
-    (property "Footprint" "" (at 134.62 92.71 0)
+    (property "Footprint" "Capacitor_SMD:C_0603_1608Metric" (at 134.62 92.71 0)
       (effects (font (size 1.27 1.27)) hide)
     )
@@
       (effects (font (size 1.27 1.27)) (justify left))
     )
-    (property "Footprint" "" (at 146.05 135.89 0)
+    (property "Footprint" "Capacitor_SMD:C_0603_1608Metric" (at 146.05 135.89 0)
       (effects (font (size 1.27 1.27)) hide)
     )
@@
       (effects (font (size 1.27 1.27)) (justify left))
     )
-    (property "Footprint" "" (at 101.6 116.84 0)
+    (property "Footprint" "Capacitor_SMD:C_0603_1608Metric" (at 101.6 116.84 0)
       (effects (font (size 1.27 1.27)) hide)
     )
@@
       (effects (font (size 1.27 1.27)) (justify left))
     )
-    (property "Footprint" "" (at 146.05 92.71 0)
-      (effects (font (size 1.27 1.27)) hide)
-    )
+    (property "Footprint" "Capacitor_SMD:C_0603_1608Metric" (at 146.05 92.71 0)
+      (effects (font (size 1.27 1.27)) hide)
+    )

Commit message: Completed schematics
Parts:
- C405, C406: footprint Capacitor_SMD:C_0603_1608Metric -> Capacitor_SMD:CP_Elec_5x5.4
- J401, J402: footprint (none) -> Connector_JST:JST_XH_S6B-XH-A_1x06_P2.50mm_Horizontal
- U401: value ZXBM5210-S -> ZXBM5210-S_1; footprint Package_SO:SOIC-8_3.9x4.9mm_P1.27mm -> Package_SO:SOIC-8-1EP_3.9x4.9mm_P1.27mm_EP2.62x3.51mm
- U402: value ZXBM5210-S -> ZXBM5210-S_2; footprint Package_SO:SOIC-8_3.9x4.9mm_P1.27mm -> Package_SO:SOIC-8-1EP_3.9x4.9mm_P1.27mm_EP2.62x3.51mm
Changed lines of the file:
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@@
       (effects (font (size 1.27 1.27)) (justify left))
     )
-    (property "Footprint" "" (at 203.2 130.81 0)
+    (property "Footprint" "Connector_JST:JST_XH_S6B-XH-A_1x06_P2.50mm_Horizontal" (at 203.2 130.81 0)
       (effects (font (size 1.27 1.27)) hide)
     )
@@
       (effects (font (size 1.27 1.27)) (justify left))
     )
-    (property "Footprint" "Capacitor_SMD:C_0603_1608Metric" (at 137.16 74.93 0)
+    (property "Footprint" "Capacitor_SMD:CP_Elec_5x5.4" (at 137.16 74.93 0)
       (effects (font (size 1.27 1.27)) hide)
     )
@@
       (effects (font (size 1.27 1.27)) (justify left))
     )
-    (property "Value" "ZXBM5210-S" (at 106.68 135.89 0)
-      (effects (font (size 1.27 1.27)) (justify left))
-    )
-    (property "Footprint" "Package_SO:SOIC-8_3.9x4.9mm_P1.27mm" (at 123.19 134.62 0)
+    (property "Value" "ZXBM5210-S_2" (at 106.68 135.89 0)
+      (effects (font (size 1.27 1.27)) (justify left))
+    )
+    (property "Footprint" "Package_SO:SOIC-8-1EP_3.9x4.9mm_P1.27mm_EP2.62x3.51mm" (at 123.19 134.62 0)
       (effects (font (size 1.27 1.27)) hide)
     )
@@
       (effects (font (size 1.27 1.27)) (justify left))
     )
-    (property "Footprint" "Capacitor_SMD:C_0603_1608Metric" (at 137.16 118.11 0)
+    (property "Footprint" "Capacitor_SMD:CP_Elec_5x5.4" (at 137.16 118.11 0)
       (effects (font (size 1.27 1.27)) hide)
     )
@@
       (effects (font (size 1.27 1.27)) (justify left))
     )
-    (property "Footprint" "" (at 203.2 87.63 0)
+    (property "Footprint" "Connector_JST:JST_XH_S6B-XH-A_1x06_P2.50mm_Horizontal" (at 203.2 87.63 0)
       (effects (font (size 1.27 1.27)) hide)
     )
@@
       (effects (font (size 1.27 1.27)) (justify left))
     )
-    (property "Value" "ZXBM5210-S" (at 106.68 92.71 0)
-      (effects (font (size 1.27 1.27)) (justify left))
-    )
-    (property "Footprint" "Package_SO:SOIC-8_3.9x4.9mm_P1.27mm" (at 123.19 91.44 0)
-      (effects (font (size 1.27 1.27)) hide)
-    )
+    (property "Value" "ZXBM5210-S_1" (at 106.68 92.71 0)
+      (effects (font (size 1.27 1.27)) (justify left))
+    )
+    (property "Footprint" "Package_SO:SOIC-8-1EP_3.9x4.9mm_P1.27mm_EP2.62x3.51mm" (at 123.19 91.44 0)
+      (effects (font (size 1.27 1.27)) hide)
+    )

Commit message: PCB finalized
Parts:
- U401, U402: footprint Package_SO:SOIC-8-1EP_3.9x4.9mm_P1.27mm_EP2.62x3.51mm -> Package_SO:SOIC-8-1EP_3.9x4.9mm_P1.27mm_EP2.514x3.2mm_ThermalVias; symbol Driver_Motor:ZXBM5210-S -> Driver_Motor:ZXBM5210-SP
Connections:
- net GND: now also U401.9 (GND), U402.9 (GND)
- net MOT2_OUT1: now reaches C404.1, J402.1 (Pin_1), U402.1 (OUT1)
- net MOT2_OUT2: now reaches C408.1, J402.6 (Pin_6), U402.7 (OUT2)
- net MOT1_OUT1: now reaches C403.1, J401.1 (Pin_1), U401.1 (OUT1)
- net MOT1_OUT2: now reaches C407.1, J401.6 (Pin_6), U401.7 (OUT2)
Changed lines of the file:
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@@
+    (effects (font (size 1.27 1.27)) (justify left bottom))
+  )
+  (label "MOT2_OUT1" (at 182.88 125.73 0) (fields_autoplaced)
+    (effects (font (size 1.27 1.27)) (justify left bottom))
+  )
+  (label "MOT1_OUT2" (at 181.61 95.25 0) (fields_autoplaced)
+    (effects (font (size 1.27 1.27)) (justify left bottom))
+  )
+  (label "MOT1_OUT1" (at 181.61 82.55 0) (fields_autoplaced)
+    (effects (font (size 1.27 1.27)) (justify left bottom))
+  )
+  (label "MOT2_OUT2" (at 182.88 138.43 0) (fields_autoplaced)
     (effects (font (size 1.27 1.27)) (justify left bottom))
   )
@@
     )
   )
-  (symbol (lib_id "Driver_Motor:ZXBM5210-S") (at 121.92 128.27 0) (unit 1)
+  (symbol (lib_id "Driver_Motor:ZXBM5210-SP") (at 121.92 128.27 0) (unit 1)
     (in_bom yes) (on_board yes) (dnp no)
     (property "Reference" "U402" (at 124.1141 135.89 0)
@@
       (effects (font (size 1.27 1.27)) (justify left))
     )
-    (property "Footprint" "Package_SO:SOIC-8-1EP_3.9x4.9mm_P1.27mm_EP2.62x3.51mm" (at 123.19 134.62 0)
+    (property "Footprint" "Package_SO:SOIC-8-1EP_3.9x4.9mm_P1.27mm_EP2.514x3.2mm_ThermalVias" (at 123.19 134.62 0)
       (effects (font (size 1.27 1.27)) hide)
     )
@@
     (pin "7")
     (pin "8")
+    (pin "9")
     (instances
       (project "kicad_chat-souris"
@@
     )
   )
-  (symbol (lib_id "Driver_Motor:ZXBM5210-S") (at 121.92 85.09 0) (unit 1)
+  (symbol (lib_id "Driver_Motor:ZXBM5210-SP") (at 121.92 85.09 0) (unit 1)
     (in_bom yes) (on_board yes) (dnp no)
     (property "Reference" "U401" (at 124.1141 92.71 0)
@@
       (effects (font (size 1.27 1.27)) (justify left))
     )
-    (property "Footprint" "Package_SO:SOIC-8-1EP_3.9x4.9mm_P1.27mm_EP2.62x3.51mm" (at 123.19 91.44 0)
+    (property "Footprint" "Package_SO:SOIC-8-1EP_3.9x4.9mm_P1.27mm_EP2.514x3.2mm_ThermalVias" (at 123.19 91.44 0)
       (effects (font (size 1.27 1.27)) hide)
     )
@@
     (pin "7")
     (pin "8")
-    (instances
-      (project "kicad_chat-souris"
+    (pin "9")
+    (instances
+      (project "kicad_chat-souris"
