File: KICAD/sensors.kicad_sch (KiCad schematic)
At the start: 16 parts, among them J401 Conn_01x02, J402 Conn_01x02, J404 Conn_01x02, J405 Conn_01x02, J501 Conn_01x08, U501 MPU-6050

Commit message: update schematics
Parts:
- C501, C502, C503, C504: footprint (none) -> Capacitor_SMD:C_0603_1608Metric
Changed lines of the file:
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@@
       (effects (font (size 1.27 1.27)) (justify left))
     )
-    (property "Footprint" "" (at 238.76 59.69 0)
+    (property "Footprint" "Capacitor_SMD:C_0603_1608Metric" (at 238.76 59.69 0)
       (effects (font (size 1.27 1.27)) hide)
     )
@@
       (effects (font (size 1.27 1.27)))
     )
-    (property "Footprint" "" (at 226.06 26.67 0)
+    (property "Footprint" "Capacitor_SMD:C_0603_1608Metric" (at 226.06 26.67 0)
       (effects (font (size 1.27 1.27)) hide)
     )
@@
       (effects (font (size 1.27 1.27)))
     )
-    (property "Footprint" "" (at 210.82 26.67 0)
+    (property "Footprint" "Capacitor_SMD:C_0603_1608Metric" (at 210.82 26.67 0)
       (effects (font (size 1.27 1.27)) hide)
     )
@@
       (effects (font (size 1.27 1.27)) (justify left))
     )
-    (property "Footprint" "" (at 248.92 59.69 0)
-      (effects (font (size 1.27 1.27)) hide)
-    )
+    (property "Footprint" "Capacitor_SMD:C_0603_1608Metric" (at 248.92 59.69 0)
+      (effects (font (size 1.27 1.27)) hide)
+    )

Commit message: Completed schematics
Parts:
- J401: value Conn_01x02 -> Conn_Bmp_1; footprint (none) -> Connector_JST:JST_XH_S2B-XH-A_1x02_P2.50mm_Horizontal
- J402: value Conn_01x02 -> Conn_Bmp_2; footprint (none) -> Connector_JST:JST_XH_S2B-XH-A_1x02_P2.50mm_Horizontal
- J404: value Conn_01x02 -> Conn_Bmp_3; footprint (none) -> Connector_JST:JST_XH_S2B-XH-A_1x02_P2.50mm_Horizontal
- J405: value Conn_01x02 -> Conn_Bmp_4; footprint (none) -> Connector_JST:JST_XH_S2B-XH-A_1x02_P2.50mm_Horizontal
- J501: value Conn_01x08 -> Conn_lidar; footprint (none) -> Connector_JST:JST_XH_S8B-XH-A_1x08_P2.50mm_Horizontal
- R401, R402, R404, R405, R505, R506: footprint (none) -> Resistor_SMD:R_0603_1608Metric
Changed lines of the file:
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@@
       (effects (font (size 1.27 1.27)) (justify right))
     )
-    (property "Value" "Conn_01x02" (at 34.29 76.2 90)
+    (property "Value" "Conn_Bmp_2" (at 34.29 76.2 90)
       (effects (font (size 1.27 1.27)) (justify right))
     )
-    (property "Footprint" "" (at 36.83 78.74 0)
+    (property "Footprint" "Connector_JST:JST_XH_S2B-XH-A_1x02_P2.50mm_Horizontal" (at 36.83 78.74 0)
       (effects (font (size 1.27 1.27)) hide)
     )
@@
       (effects (font (size 1.27 1.27)) (justify right))
     )
-    (property "Value" "Conn_01x02" (at 81.28 49.53 90)
+    (property "Value" "Conn_Bmp_3" (at 81.28 49.53 90)
       (effects (font (size 1.27 1.27)) (justify right))
     )
-    (property "Footprint" "" (at 83.82 52.07 0)
+    (property "Footprint" "Connector_JST:JST_XH_S2B-XH-A_1x02_P2.50mm_Horizontal" (at 83.82 52.07 0)
       (effects (font (size 1.27 1.27)) hide)
     )
@@
       (effects (font (size 1.27 1.27)))
     )
-    (property "Footprint" "" (at 275.59 41.91 0)
+    (property "Footprint" "Resistor_SMD:R_0603_1608Metric" (at 275.59 41.91 0)
       (effects (font (size 1.27 1.27)) hide)
     )
@@
       (effects (font (size 1.27 1.27)) (justify right))
     )
-    (property "Value" "Conn_01x02" (at 81.28 76.2 90)
+    (property "Value" "Conn_Bmp_4" (at 81.28 76.2 90)
       (effects (font (size 1.27 1.27)) (justify right))
     )
-    (property "Footprint" "" (at 83.82 78.74 0)
+    (property "Footprint" "Connector_JST:JST_XH_S2B-XH-A_1x02_P2.50mm_Horizontal" (at 83.82 78.74 0)
       (effects (font (size 1.27 1.27)) hide)
     )
@@
       (effects (font (size 1.27 1.27)) (justify left))
     )
-    (property "Footprint" "" (at 49.53 54.61 0)
+    (property "Footprint" "Resistor_SMD:R_0603_1608Metric" (at 49.53 54.61 0)
       (effects (font (size 1.27 1.27)) hide)
     )
@@
       (effects (font (size 1.27 1.27)) (justify right))
     )
-    (property "Value" "Conn_01x02" (at 34.29 49.53 90)
+    (property "Value" "Conn_Bmp_1" (at 34.29 49.53 90)
       (effects (font (size 1.27 1.27)) (justify right))
     )
-    (property "Footprint" "" (at 36.83 52.07 0)
+    (property "Footprint" "Connector_JST:JST_XH_S2B-XH-A_1x02_P2.50mm_Horizontal" (at 36.83 52.07 0)
       (effects (font (size 1.27 1.27)) hide)
     )
@@
       (effects (font (size 1.27 1.27)) (justify left))
     )
-    (property "Footprint" "" (at 96.52 81.28 0)
+    (property "Footprint" "Resistor_SMD:R_0603_1608Metric" (at 96.52 81.28 0)
       (effects (font (size 1.27 1.27)) hide)
     )
@@
   (symbol (lib_id "Connector_Generic:Conn_01x08") (at 66.04 114.3 0) (unit 1)
     (in_bom yes) (on_board yes) (dnp no) (fields_autoplaced)
-    (property "Reference" "J501" (at 72.39 115.57 90)
-      (effects (font (size 1.27 1.27)))
-    )
-    (property "Value" "Conn_01x08" (at 69.85 115.57 90)
-      (effects (font (size 1.27 1.27)))
-    )
-    (property "Footprint" "" (at 66.04 114.3 0)
+    (property "Reference" "J501" (at 68.58 114.3 0)
+      (effects (font (size 1.27 1.27)) (justify left))
+    )
+    (property "Value" "Conn_lidar" (at 68.58 116.84 0)
+      (effects (font (size 1.27 1.27)) (justify left))
+    )
+    (property "Footprint" "Connector_JST:JST_XH_S8B-XH-A_1x08_P2.50mm_Horizontal" (at 66.04 114.3 0)
       (effects (font (size 1.27 1.27)) hide)
     )
@@
       (effects (font (size 1.27 1.27)) (justify left))
     )
-    (property "Footprint" "" (at 96.52 54.61 0)
+    (property "Footprint" "Resistor_SMD:R_0603_1608Metric" (at 96.52 54.61 0)
       (effects (font (size 1.27 1.27)) hide)
     )
@@
       (effects (font (size 1.27 1.27)) (justify left))
     )
-    (property "Footprint" "" (at 49.53 81.28 0)
+    (property "Footprint" "Resistor_SMD:R_0603_1608Metric" (at 49.53 81.28 0)
       (effects (font (size 1.27 1.27)) hide)
     )
@@
       (effects (font (size 1.27 1.27)))
     )
-    (property "Footprint" "" (at 266.7 41.91 0)
-      (effects (font (size 1.27 1.27)) hide)
-    )
+    (property "Footprint" "Resistor_SMD:R_0603_1608Metric" (at 266.7 41.91 0)
+      (effects (font (size 1.27 1.27)) hide)
+    )

Commit message: PCB finalized
Parts:
- added C505: 4.7µ, Capacitor_SMD:CP_Elec_5x5.4, symbol Device:C_Polarized
- added J305: SCL, Connector_PinHeader_2.54mm:PinHeader_1x01_P2.54mm_Vertical, symbol Connector:Conn_01x01_Pin
- added J305: SDA, Connector_PinHeader_2.54mm:PinHeader_1x01_P2.54mm_Vertical, symbol Connector:Conn_01x01_Pin
Connections:
- net +3.3V is gone; now on net +3V3: R401.2, R402.2, R404.2, R405.2
- net +5V: now also C505.1
- net GND: now also C505.2
- net IMU_SCL: now also J305.1 (Pin_1)
- net IMU_SDA: now also J305.1 (Pin_1)
